File: mcu.kicad_sch (KiCad schematic)
At the start: 17 parts, among them SW301 SW_Push, U203 STM32F103C8Tx, U301 M95640-WMN6TP, Y301 12MHz

Commit message: Finish PCB
Connections:
- net DIRECTION: now also U203.4 (PC15-OSC32_OUT); no longer U203.2 (PC13-TAMPER-RTC)
- net DIRECTION1: now also U203.10 (PA0-WKUP); no longer U203.21 (PB10)
- net DIRECTION2: now also U203.11 (PA1); no longer U203.22 (PB11)
- net ENABLE_LEFT: now also U203.21 (PB10); no longer U203.11 (PA1)
- net ENABLE_RIGHT: now also U203.22 (PB11); no longer U203.10 (PA0-WKUP)
- net IO1: now also U203.18 (PB0); no longer U203.16 (PA6)
- net IO3: now also U203.16 (PA6); no longer U203.18 (PB0)
- net PWM_LEFT: now also U203.31 (PA10); no longer U203.29 (PA8)
- net PWM_RIGHT: now also U203.29 (PA8); no longer U203.31 (PA10)
- net STEER_LOCK_RIGHT: now also U203.2 (PC13-TAMPER-RTC); no longer U203.4 (PC15-OSC32_OUT)
- net TEMP_LEFT: now also U203.15 (PA5); no longer U203.14 (PA4)
- net TEMP_RIGHT: now also U203.14 (PA4); no longer U203.15 (PA5)
- net D-: now reaches R303.1, U203.32 (PA11)
- net D+: now reaches R304.1, U203.33 (PA12)
- net USB_DM renamed USB_DN
Changed lines of the file:
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@@
     (effects (font (size 1.27 1.27)) (justify left bottom))
+  )
+  (label "D-" (at 130.81 95.25 180)
+    (effects (font (size 1.27 1.27)) (justify right bottom))
+  )
+  (label "D+" (at 130.81 97.79 180)
+    (effects (font (size 1.27 1.27)) (justify right bottom))
   )
   (label "USB_PULL" (at 137.16 105.41 180)
@@
     (effects (font (size 1.27 1.27)) (justify right))
   )
-  (hierarchical_label "DIRECTION1" (shape output) (at 72.39 92.71 180)
+  (hierarchical_label "ENABLE_LEFT" (shape output) (at 72.39 92.71 180)
     (effects (font (size 1.27 1.27)) (justify right))
   )
-  (hierarchical_label "DIRECTION2" (shape output) (at 72.39 95.25 180)
+  (hierarchical_label "ENABLE_RIGHT" (shape output) (at 72.39 95.25 180)
     (effects (font (size 1.27 1.27)) (justify right))
   )
-  (hierarchical_label "IO3" (shape bidirectional) (at 77.47 67.31 180)
+  (hierarchical_label "IO1" (shape bidirectional) (at 77.47 67.31 180)
     (effects (font (size 1.27 1.27)) (justify right))
   )
@@
     (effects (font (size 1.27 1.27)) (justify right))
   )
-  (hierarchical_label "DIRECTION" (shape input) (at 77.47 111.76 180)
+  (hierarchical_label "STEER_LOCK_RIGHT" (shape input) (at 77.47 111.76 180)
     (effects (font (size 1.27 1.27)) (justify right))
   )
@@
     (effects (font (size 1.27 1.27)) (justify right))
   )
-  (hierarchical_label "STEER_LOCK_RIGHT" (shape input) (at 77.47 116.84 180)
+  (hierarchical_label "DIRECTION" (shape input) (at 77.47 116.84 180)
     (effects (font (size 1.27 1.27)) (justify right))
   )
-  (hierarchical_label "PWM_LEFT" (shape output) (at 130.81 87.63 0)
+  (hierarchical_label "PWM_RIGHT" (shape output) (at 130.81 87.63 0)
     (effects (font (size 1.27 1.27)) (justify left))
   )
-  (hierarchical_label "PWM_RIGHT" (shape output) (at 130.81 92.71 0)
+  (hierarchical_label "PWM_LEFT" (shape output) (at 130.81 92.71 0)
     (effects (font (size 1.27 1.27)) (justify left))
   )
-  (hierarchical_label "TEMP_LEFT" (shape input) (at 134.62 77.47 0)
+  (hierarchical_label "TEMP_RIGHT" (shape input) (at 134.62 77.47 0)
     (effects (font (size 1.27 1.27)) (justify left))
   )
-  (hierarchical_label "TEMP_RIGHT" (shape input) (at 134.62 80.01 0)
+  (hierarchical_label "TEMP_LEFT" (shape input) (at 134.62 80.01 0)
     (effects (font (size 1.27 1.27)) (justify left))
   )
-  (hierarchical_label "IO1" (shape bidirectional) (at 134.62 82.55 0)
+  (hierarchical_label "IO3" (shape bidirectional) (at 134.62 82.55 0)
     (effects (font (size 1.27 1.27)) (justify left))
   )
@@
     (effects (font (size 1.27 1.27)) (justify left))
   )
-  (hierarchical_label "ENABLE_RIGHT" (shape output) (at 135.89 67.31 0)
+  (hierarchical_label "DIRECTION1" (shape output) (at 135.89 67.31 0)
     (effects (font (size 1.27 1.27)) (justify left))
   )
-  (hierarchical_label "ENABLE_LEFT" (shape output) (at 135.89 69.85 0)
+  (hierarchical_label "DIRECTION2" (shape output) (at 135.89 69.85 0)
     (effects (font (size 1.27 1.27)) (justify left))
   )
@@
     (effects (font (size 1.27 1.27)) (justify left))
   )
-  (hierarchical_label "USB_DM" (shape bidirectional) (at 154.94 95.25 0)
+  (hierarchical_label "USB_DN" (shape bidirectional) (at 154.94 95.25 0)
     (effects (font (size 1.27 1.27)) (justify left))
   )
