File: mcu.kicad_sch (KiCad schematic)
At the start: 17 parts, among them SW301 SW_Push, U203 STM32F103C8Tx, U301 M95640-WMN6TP, Y301 12MHz

Commit message: Tweak PCB and add gerbers
Parts:
- removed Y301: 12MHz, Crystal:Crystal_SMD_3225-4Pin_3.2x2.5mm_HandSoldering, symbol Device:Crystal_GND24
- added R310, R311, R312: 22R, Resistor_SMD:R_0603_1608Metric_Pad0.98x0.95mm_HandSolder, symbol Device:R
- added Y301: 8MHz, Crystal:Crystal_SMD_5032-2Pin_5.0x3.2mm_HandSoldering, symbol Device:Crystal
- R308, R309: value 62k -> 10k
- SW301: footprint Button_Switch_SMD:SW_SPST_TL3342 -> GozLib:SW_SPST_TS-1185EC
Connections:
- net ENABLE_LEFT: now also U203.22 (PB11); no longer U203.21 (PB10)
- net ENABLE_RIGHT: now also U203.21 (PB10); no longer U203.22 (PB11)
- net MISO: now also R312.1; no longer U203.27 (PB14)
- net MOSI: now also R311.1; no longer U203.28 (PB15)
- net SCK: now also R310.1; no longer U203.26 (PB13)
- net at C303.1, U203.5 (PD0-OSC_IN): now also Y301.2
- net at C302.1, U203.6 (PD1-OSC_IN): now also Y301.1
- new net: R310.2, U203.26 (PB13)
- new net: R312.2, U203.27 (PB14)
- new net: R311.2, U203.28 (PB15)
Changed lines of the file:
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@@
   (junction (at 144.78 124.46) (diameter 0.9144) (color 0 0 0 0))
   (junction (at 153.67 97.79) (diameter 0.9144) (color 0 0 0 0))
-  (junction (at 162.56 129.54) (diameter 0.9144) (color 0 0 0 0))
   (junction (at 176.53 90.17) (diameter 0.9144) (color 0 0 0 0))
   (junction (at 191.77 40.64) (diameter 0.9144) (color 0 0 0 0))
@@
     (stroke (width 0) (type solid) (color 0 0 0 0))
   )
+  (wire (pts (xy 63.5 100.33) (xy 72.39 100.33))
+    (stroke (width 0) (type solid) (color 0 0 0 0))
+  )
+  (wire (pts (xy 63.5 102.87) (xy 72.39 102.87))
+    (stroke (width 0) (type solid) (color 0 0 0 0))
+  )
+  (wire (pts (xy 63.5 105.41) (xy 72.39 105.41))
+    (stroke (width 0) (type solid) (color 0 0 0 0))
+  )
   (wire (pts (xy 64.77 50.8) (xy 49.53 50.8))
     (stroke (width 0) (type solid) (color 0 0 0 0))
@@
     (stroke (width 0) (type solid) (color 0 0 0 0))
   )
-  (wire (pts (xy 74.93 100.33) (xy 81.28 100.33))
-    (stroke (width 0) (type solid) (color 0 0 0 0))
-  )
-  (wire (pts (xy 74.93 102.87) (xy 81.28 102.87))
-    (stroke (width 0) (type solid) (color 0 0 0 0))
-  )
-  (wire (pts (xy 74.93 105.41) (xy 81.28 105.41))
-    (stroke (width 0) (type solid) (color 0 0 0 0))
-  )
   (wire (pts (xy 77.47 67.31) (xy 81.28 67.31))
     (stroke (width 0) (type solid) (color 0 0 0 0))
@@
     (stroke (width 0) (type solid) (color 0 0 0 0))
   )
+  (wire (pts (xy 80.01 100.33) (xy 81.28 100.33))
+    (stroke (width 0) (type solid) (color 0 0 0 0))
+  )
+  (wire (pts (xy 80.01 102.87) (xy 81.28 102.87))
+    (stroke (width 0) (type solid) (color 0 0 0 0))
+  )
+  (wire (pts (xy 80.01 105.41) (xy 81.28 105.41))
+    (stroke (width 0) (type solid) (color 0 0 0 0))
+  )
   (wire (pts (xy 81.28 60.96) (xy 74.93 60.96))
     (stroke (width 0) (type solid) (color 0 0 0 0))
@@
     (stroke (width 0) (type solid) (color 0 0 0 0))
   )
-  (wire (pts (xy 139.7 119.38) (xy 162.56 119.38))
-    (stroke (width 0) (type solid) (color 0 0 0 0))
-  )
-  (wire (pts (xy 139.7 129.54) (xy 162.56 129.54))
-    (stroke (width 0) (type solid) (color 0 0 0 0))
-  )
   (wire (pts (xy 139.7 142.24) (xy 139.7 143.51))
     (stroke (width 0) (type solid) (color 0 0 0 0))
@@
     (stroke (width 0) (type solid) (color 0 0 0 0))
   )
-  (wire (pts (xy 162.56 119.38) (xy 162.56 129.54))
-    (stroke (width 0) (type solid) (color 0 0 0 0))
-  )
-  (wire (pts (xy 162.56 129.54) (xy 162.56 132.08))
-    (stroke (width 0) (type solid) (color 0 0 0 0))
-  )
   (wire (pts (xy 185.42 40.64) (xy 191.77 40.64))
     (stroke (width 0) (type solid) (color 0 0 0 0))
@@
   (wire (pts (xy 243.84 40.64) (xy 248.92 40.64))
     (stroke (width 0) (type solid) (color 0 0 0 0))
+  )
+  (label "SCK" (at 63.5 100.33 0)
+    (effects (font (size 1.27 1.27)) (justify left bottom))
+  )
+  (label "MISO" (at 63.5 102.87 0)
+    (effects (font (size 1.27 1.27)) (justify left bottom))
+  )
+  (label "MOSI" (at 63.5 105.41 0)
+    (effects (font (size 1.27 1.27)) (justify left bottom))
   )
   (label "CS" (at 74.93 97.79 0)
     (effects (font (size 1.27 1.27)) (justify left bottom))
   )
-  (label "SCK" (at 74.93 100.33 0)
-    (effects (font (size 1.27 1.27)) (justify left bottom))
-  )
-  (label "MISO" (at 74.93 102.87 0)
-    (effects (font (size 1.27 1.27)) (justify left bottom))
-  )
-  (label "MOSI" (at 74.93 105.41 0)
-    (effects (font (size 1.27 1.27)) (justify left bottom))
-  )
   (label "D-" (at 130.81 95.25 180)
     (effects (font (size 1.27 1.27)) (justify right bottom))
@@
     (effects (font (size 1.27 1.27)) (justify left bottom))
   )
-  (label "SCK" (at 226.06 35.56 180)
+  (label "SCK" (at 227.33 35.56 180)
     (effects (font (size 1.27 1.27)) (justify right bottom))
   )
-  (label "MOSI" (at 226.06 38.1 180)
+  (label "MOSI" (at 227.33 38.1 180)
     (effects (font (size 1.27 1.27)) (justify right bottom))
   )
-  (label "MISO" (at 226.06 40.64 180)
+  (label "MISO" (at 227.33 40.64 180)
     (effects (font (size 1.27 1.27)) (justify right bottom))
   )
@@
     (effects (font (size 1.27 1.27)) (justify right))
   )
-  (hierarchical_label "ENABLE_LEFT" (shape output) (at 72.39 92.71 180)
-    (effects (font (size 1.27 1.27)) (justify right))
-  )
-  (hierarchical_label "ENABLE_RIGHT" (shape output) (at 72.39 95.25 180)
+  (hierarchical_label "ENABLE_RIGHT" (shape output) (at 72.39 92.71 180)
+    (effects (font (size 1.27 1.27)) (justify right))
+  )
+  (hierarchical_label "ENABLE_LEFT" (shape output) (at 72.39 95.25 180)
     (effects (font (size 1.27 1.27)) (justify right))
   )
@@
     (pin "1")
   )
-  (symbol (lib_id "power:GND") (at 162.56 132.08 0) (unit 1)
-    (in_bom yes) (on_board yes) (fields_autoplaced)
-    (property "Reference" "#PWR0306" (id 0) (at 162.56 138.43 0)
-      (effects (font (size 1.27 1.27)) hide)
-    )
-    (property "Value" "GND" (id 1) (at 162.56 137.16 0))
-    (property "Footprint" "" (id 2) (at 162.56 132.08 0)
-      (effects (font (size 1.27 1.27)) hide)
-    )
-    (property "Datasheet" "" (id 3) (at 162.56 132.08 0)
-      (effects (font (size 1.27 1.27)) hide)
-    )
-    (pin "1")
-  )
   (symbol (lib_id "power:GND") (at 176.53 97.79 0) (unit 1)
     (in_bom yes) (on_board yes) (fields_autoplaced)
@@
     )
     (property "Datasheet" "~" (id 3) (at 74.93 44.45 0)
+      (effects (font (size 1.27 1.27)) hide)
+    )
+    (pin "1")
+    (pin "2")
+  )
+  (symbol (lib_id "Device:R") (at 76.2 100.33 90) (unit 1)
+    (in_bom yes) (on_board yes)
+    (property "Reference" "R310" (id 0) (at 71.12 99.06 90))
+    (property "Value" "22R" (id 1) (at 76.2 100.33 90))
+    (property "Footprint" "Resistor_SMD:R_0603_1608Metric_Pad0.98x0.95mm_HandSolder" (id 2) (at 76.2 102.108 90)
+      (effects (font (size 1.27 1.27)) hide)
+    )
+    (property "Datasheet" "~" (id 3) (at 76.2 100.33 0)
+      (effects (font (size 1.27 1.27)) hide)
+    )
+    (pin "1")
+    (pin "2")
+  )
+  (symbol (lib_id "Device:R") (at 76.2 102.87 90) (unit 1)
+    (in_bom yes) (on_board yes)
+    (property "Reference" "R312" (id 0) (at 71.12 101.6 90))
+    (property "Value" "22R" (id 1) (at 76.2 102.87 90))
+    (property "Footprint" "Resistor_SMD:R_0603_1608Metric_Pad0.98x0.95mm_HandSolder" (id 2) (at 76.2 104.648 90)
+      (effects (font (size 1.27 1.27)) hide)
+    )
+    (property "Datasheet" "~" (id 3) (at 76.2 102.87 0)
+      (effects (font (size 1.27 1.27)) hide)
+    )
+    (pin "1")
+    (pin "2")
+  )
+  (symbol (lib_id "Device:R") (at 76.2 105.41 90) (unit 1)
+    (in_bom yes) (on_board yes)
+    (property "Reference" "R311" (id 0) (at 71.12 104.14 90))
+    (property "Value" "22R" (id 1) (at 76.2 105.41 90))
+    (property "Footprint" "Resistor_SMD:R_0603_1608Metric_Pad0.98x0.95mm_HandSolder" (id 2) (at 76.2 107.188 90)
+      (effects (font (size 1.27 1.27)) hide)
+    )
+    (property "Datasheet" "~" (id 3) (at 76.2 105.41 0)
       (effects (font (size 1.27 1.27)) hide)
     )
@@
       (effects (font (size 1.27 1.27)) (justify left))
     )
-    (property "Value" "62k" (id 1) (at 185.42 36.8299 0)
+    (property "Value" "10k" (id 1) (at 185.42 36.8299 0)
       (effects (font (size 1.27 1.27)) (justify left))
     )
@@
       (effects (font (size 1.27 1.27)) (justify left))
     )
-    (property "Value" "62k" (id 1) (at 245.11 46.9899 0)
+    (property "Value" "10k" (id 1) (at 245.11 46.9899 0)
       (effects (font (size 1.27 1.27)) (justify left))
     )
@@
       (effects (font (size 1.27 1.27)) (justify right))
     )
-    (property "Footprint" "Button_Switch_SMD:SW_SPST_TL3342" (id 2) (at 44.45 55.88 0)
+    (property "Footprint" "GozLib:SW_SPST_TS-1185EC" (id 2) (at 44.45 55.88 0)
       (effects (font (size 1.27 1.27)) hide)
     )
@@
     (pin "2")
   )
-  (symbol (lib_id "Device:Crystal_GND24") (at 139.7 124.46 0) (unit 1)
-    (in_bom yes) (on_board yes) (fields_autoplaced)
-    (property "Reference" "Y301" (id 0) (at 144.78 123.1899 0)
-      (effects (font (size 1.27 1.27)) (justify left))
-    )
-    (property "Value" "12MHz" (id 1) (at 144.78 125.7299 0)
-      (effects (font (size 1.27 1.27)) (justify left))
-    )
-    (property "Footprint" "Crystal:Crystal_SMD_3225-4Pin_3.2x2.5mm_HandSoldering" (id 2) (at 139.7 124.46 0)
+  (symbol (lib_id "Device:Crystal") (at 139.7 124.46 0) (unit 1)
+    (in_bom yes) (on_board yes) (fields_autoplaced)
+    (property "Reference" "Y301" (id 0) (at 139.7 116.84 0))
+    (property "Value" "8MHz" (id 1) (at 139.7 119.38 0))
+    (property "Footprint" "Crystal:Crystal_SMD_5032-2Pin_5.0x3.2mm_HandSoldering" (id 2) (at 139.7 124.46 0)
       (effects (font (size 1.27 1.27)) hide)
     )
@@
     (pin "1")
     (pin "2")
-    (pin "3")
-    (pin "4")
   )
   (symbol (lib_id "GozLib:M95640-WMN6TP") (at 209.55 38.1 0) (unit 1)
