File: motorcontroller.kicad_pcb (KiCad board)
At the start: 0 parts

Commit message: Start PCB
Parts:
- added BZ101: PS1240P02BT, Buzzer_Beeper:Buzzer_TDK_PS1240P02BT_D12.2mm_H6.5mm, F.Cu at (15.7, 137.0)
- added C101: 100nF, Capacitor_SMD:C_0805_2012Metric_Pad1.18x1.45mm_HandSolder, F.Cu at (27.0, 156.0)
- added C201: 100uF, Capacitor_SMD:CP_Elec_10x10.5, F.Cu at (99.2, 108.0)
- added C202: 470uF, Capacitor_SMD:CP_Elec_10x10, F.Cu at (76.0, 98.0)
- added C203: 100nF, Capacitor_SMD:C_0805_2012Metric_Pad1.18x1.45mm_HandSolder, F.Cu at (121.0, 107.0)
- added C204: 1uF, Capacitor_SMD:C_0805_2012Metric_Pad1.18x1.45mm_HandSolder, F.Cu at (111.0, 141.0)
- added C205: 2200uF, Capacitor_THT:CP_Radial_D16.0mm_P7.50mm, F.Cu at (63.5, 34.0)
- added C206: 2200uF, Capacitor_THT:CP_Radial_D16.0mm_P7.50mm, F.Cu at (70.5, 50.0)
- added C207: 2200uF, Capacitor_THT:CP_Radial_D16.0mm_P7.50mm, F.Cu at (63.5, 66.0)
- added C208: 2200uF, Capacitor_THT:CP_Radial_D16.0mm_P7.50mm, F.Cu at (70.5, 82.0)
- added C209: 100nF, Capacitor_SMD:C_0805_2012Metric_Pad1.18x1.45mm_HandSolder, F.Cu at (126.0, 107.0)
- added C210: 1mF, Capacitor_THT:CP_Radial_D10.0mm_P5.00mm, F.Cu at (61.6, 92.0)
- added C211: 330uF, Capacitor_SMD:CP_Elec_6.3x5.4, F.Cu at (88.0, 100.0)
- added C212: 1nF, Capacitor_SMD:C_0805_2012Metric_Pad1.18x1.45mm_HandSolder, F.Cu at (138.0, 111.0)
- added C213: 1uF, Capacitor_SMD:C_0805_2012Metric_Pad1.18x1.45mm_HandSolder, F.Cu at (68.0, 169.0)
- added C214: 10nF, Capacitor_SMD:C_0805_2012Metric_Pad1.18x1.45mm_HandSolder, F.Cu at (68.0, 164.0)
- added C215: 100nF, Capacitor_SMD:C_0805_2012Metric_Pad1.18x1.45mm_HandSolder, F.Cu at (67.0, 158.0)
- added C216: 100nF, Capacitor_SMD:C_0805_2012Metric_Pad1.18x1.45mm_HandSolder, F.Cu at (73.0, 158.0)
- added C217: 100nF, Capacitor_SMD:C_0805_2012Metric_Pad1.18x1.45mm_HandSolder, F.Cu at (73.0, 162.0)
- added C218: 10nF, Capacitor_SMD:C_0805_2012Metric_Pad1.18x1.45mm_HandSolder, F.Cu at (68.0, 183.0)
- added C219: 100nF, Capacitor_SMD:C_0805_2012Metric_Pad1.18x1.45mm_HandSolder, F.Cu at (73.0, 166.0)
- added C220: 4.7uF, Capacitor_SMD:C_0805_2012Metric_Pad1.18x1.45mm_HandSolder, F.Cu at (73.0, 170.0)
- added C301: 100nF, Capacitor_SMD:C_0805_2012Metric_Pad1.18x1.45mm_HandSolder, F.Cu at (73.0, 182.0)
- added C302: 20pF, Capacitor_SMD:C_0805_2012Metric_Pad1.18x1.45mm_HandSolder, F.Cu at (56.0, 151.0)
- added C303: 20pF, Capacitor_SMD:C_0805_2012Metric_Pad1.18x1.45mm_HandSolder, F.Cu at (56.0, 148.0)
- added C304: 100nF, Capacitor_SMD:C_0805_2012Metric_Pad1.18x1.45mm_HandSolder, F.Cu at (28.0, 176.3)
- added C401: 1uF, Capacitor_SMD:C_0805_2012Metric_Pad1.18x1.45mm_HandSolder, F.Cu at (38.0, 48.5)
- added C402: 100nF, Capacitor_SMD:C_0805_2012Metric_Pad1.18x1.45mm_HandSolder, F.Cu at (37.0, 38.5)
- added C403: 1uF, Capacitor_SMD:C_0805_2012Metric_Pad1.18x1.45mm_HandSolder, F.Cu at (38.0, 87.5)
- added C404: 100nF, Capacitor_SMD:C_0805_2012Metric_Pad1.18x1.45mm_HandSolder, F.Cu at (38.0, 78.5)
- added C405: 10nF, Capacitor_SMD:C_0805_2012Metric_Pad1.18x1.45mm_HandSolder, F.Cu at (21.0, 65.5)
- added C406: 10nF, Capacitor_SMD:C_0805_2012Metric_Pad1.18x1.45mm_HandSolder, F.Cu at (118.0, 65.0)
- added C407: 1uF, Capacitor_SMD:C_0805_2012Metric_Pad1.18x1.45mm_HandSolder, F.Cu at (103.0, 49.0)
- added C408: 100nF, Capacitor_SMD:C_0805_2012Metric_Pad1.18x1.45mm_HandSolder, F.Cu at (103.0, 38.0)
- added C409: 1uF, Capacitor_SMD:C_0805_2012Metric_Pad1.18x1.45mm_HandSolder, F.Cu at (103.0, 78.0)
- added C410: 100nF, Capacitor_SMD:C_0805_2012Metric_Pad1.18x1.45mm_HandSolder, F.Cu at (103.0, 87.0)
- added D101: PWR, LED_SMD:LED_0805_2012Metric_Pad1.15x1.40mm_HandSolder, F.Cu at (103.0, 122.0)
- added D102: LED1, LED_SMD:LED_0805_2012Metric_Pad1.15x1.40mm_HandSolder, F.Cu at (35.0, 111.0)
- added D103: LED2, LED_SMD:LED_0805_2012Metric_Pad1.15x1.40mm_HandSolder, F.Cu at (31.0, 111.0)
- added D201: PMEG3030EP,115, Diode_SMD:D_SOD-128, F.Cu at (103.8, 132.0)
- added D202: PMEG3030EP,115, Diode_SMD:D_SOD-128, F.Cu at (103.8, 137.0)
- added D203: SK32, Diode_SMD:D_SOD-123F, F.Cu at (121.0, 119.0)
- added D204: SK32, Diode_SMD:D_SOD-123F, F.Cu at (116.0, 141.0)
- added D401: G30C120CTW, Package_TO_SOT_THT:TO-220-3_Vertical, F.Cu at (30.0, 41.0)
- added D402: G30C120CTW, Package_TO_SOT_THT:TO-220-3_Vertical, F.Cu at (30.0, 80.0)
- added D403: G30C120CTW, Package_TO_SOT_THT:TO-220-3_Vertical, F.Cu at (110.9, 46.5)
- added D404: G30C120CTW, Package_TO_SOT_THT:TO-220-3_Vertical, F.Cu at (110.9, 85.5)
- added D501: SS210, Diode_SMD:D_SMA_Handsoldering, F.Cu at (103.1, 157.9)
- added D502: SS210, Diode_SMD:D_SMA_Handsoldering, F.Cu at (103.1, 162.9)
- added D503: SS210, Diode_SMD:D_SMA_Handsoldering, F.Cu at (103.1, 167.9)
- added D504: SS210, Diode_SMD:D_SMA_Handsoldering, F.Cu at (102.6, 171.9)
- added F201: Fuse, Fuse:Fuseholder_Littelfuse_Nano2_154x, F.Cu at (123.8, 113.0)
- added H101: MountingHole, MountingHole:MountingHole_4.3mm_M4, F.Cu at (38.0, 30.0)
- added H102: MountingHole, MountingHole:MountingHole_4.3mm_M4, F.Cu at (103.0, 30.0)
- added H103: MountingHole, MountingHole:MountingHole_4.3mm_M4, F.Cu at (32.0, 121.0)
- added H104: MountingHole, MountingHole:MountingHole_4.3mm_M4, F.Cu at (109.0, 121.0)
- added H105: MountingHole_Pad, MountingHole:MountingHole_4.3mm_M4_Pad, F.Cu at (50.5, 88.0)
- added H106: MountingHole_Pad, MountingHole:MountingHole_4.3mm_M4_Pad, F.Cu at (90.5, 88.0)
- added H107: MountingHole_Pad, MountingHole:MountingHole_4.3mm_M4_Pad, F.Cu at (50.5, 61.0)
- added H108: MountingHole_Pad, MountingHole:MountingHole_4.3mm_M4_Pad, F.Cu at (90.5, 61.0)
- added H109: MountingHole_Pad, MountingHole:MountingHole_4.3mm_M4_Pad, F.Cu at (50.5, 35.0)
- added H110: MountingHole_Pad, MountingHole:MountingHole_4.3mm_M4_Pad, F.Cu at (90.5, 35.0)
- added J101: TYPE-C-31-M-12, Connector_USB:USB_C_Receptacle_HRO_TYPE-C-31-M-12, F.Cu at (44.0, 121.0)
- added J102: STLink_02x05, Connector_PinHeader_2.54mm:PinHeader_2x05_P2.54mm_Vertical, F.Cu at (58.0, 107.0)
- added J103: STRLCK, Connector_JST:JST_XH_B3B-XH-A_1x03_P2.50mm_Vertical, F.Cu at (63.0, 121.5)
- added J104: IGN, Connector_JST:JST_XH_B3B-XH-A_1x03_P2.50mm_Vertical, F.Cu at (81.5, 121.5)
- added J105: THROTTLE, Connector_JST:JST_XH_B3B-XH-A_1x03_P2.50mm_Vertical, F.Cu at (72.0, 121.5)
- added J106: UART, Connector_PinHeader_2.54mm:PinHeader_1x03_P2.54mm_Vertical, F.Cu at (32.0, 105.0)
- added J107: IO, Connector_PinHeader_2.54mm:PinHeader_1x08_P2.54mm_Vertical, F.Cu at (41.9, 101.0)
- added J108: DIR, Connector_JST:JST_XH_B2B-XH-A_1x02_P2.50mm_Vertical, F.Cu at (69.0, 109.0)
- added J109: EN, Connector_JST:JST_XH_B2B-XH-A_1x02_P2.50mm_Vertical, F.Cu at (81.0, 108.0)
- added J110: CAN, Connector_JST:JST_XH_B3B-XH-A_1x03_P2.50mm_Vertical, F.Cu at (53.5, 121.5)
- added J201: FUSE, Connector_JST:JST_XH_B2B-XH-A_1x02_P2.50mm_Vertical, F.Cu at (97.0, 121.0)
- added L201: 47uH, Resistor_SMD:R_0805_2012Metric_Pad1.20x1.40mm_HandSolder, F.Cu at (127.0, 119.0)
- added L202: 47uH, Resistor_SMD:R_0805_2012Metric_Pad1.20x1.40mm_HandSolder, F.Cu at (111.0, 145.0)
- added L203: FCM2012KF-601T05, Resistor_SMD:R_0805_2012Metric_Pad1.20x1.40mm_HandSolder, F.Cu at (61.0, 174.0)
- added Q101: AP2300, Package_TO_SOT_SMD:TSOT-23_HandSoldering, F.Cu at (30.0, 137.0)
- added Q401: STP15810, Package_TO_SOT_THT:TO-220-3_Vertical, F.Cu at (30.0, 30.0)
- added Q402: STP15810, Package_TO_SOT_THT:TO-220-3_Vertical, F.Cu at (30.0, 52.0)
- added Q403: STP15810, Package_TO_SOT_THT:TO-220-3_Vertical, F.Cu at (30.0, 69.0)
- added Q404: STP15810, Package_TO_SOT_THT:TO-220-3_Vertical, F.Cu at (30.0, 91.0)
- added Q405: STP15810, Package_TO_SOT_THT:TO-220-3_Vertical, F.Cu at (110.9, 35.5)
- added Q406: STP15810, Package_TO_SOT_THT:TO-220-3_Vertical, F.Cu at (110.9, 57.5)
- added Q407: STP15810, Package_TO_SOT_THT:TO-220-3_Vertical, F.Cu at (110.9, 74.5)
- added Q408: STP15810, Package_TO_SOT_THT:TO-220-3_Vertical, F.Cu at (110.9, 96.5)
- added Q501: WSP6946, Package_SO:SOP-8_3.9x4.9mm_P1.27mm, F.Cu at (93.4, 179.1)
- added Q502: WSP6946, Package_SO:SOP-8_3.9x4.9mm_P1.27mm, F.Cu at (93.0, 162.0)
- added R101: 0R, Resistor_SMD:R_0603_1608Metric_Pad0.98x0.95mm_HandSolder, F.Cu at (42.0, 127.0)
- added R102: 5.1k, Resistor_SMD:R_0603_1608Metric_Pad0.98x0.95mm_HandSolder, F.Cu at (42.0, 132.0)
- added R103: 5.1k, Resistor_SMD:R_0603_1608Metric_Pad0.98x0.95mm_HandSolder, F.Cu at (42.0, 137.0)
- added R104: 10k, Resistor_SMD:R_0603_1608Metric_Pad0.98x0.95mm_HandSolder, F.Cu at (64.0, 127.0)
- added R105: 10k, Resistor_SMD:R_0603_1608Metric_Pad0.98x0.95mm_HandSolder, F.Cu at (82.0, 127.0)
- added R106: 4.7k, Resistor_SMD:R_0603_1608Metric_Pad0.98x0.95mm_HandSolder, F.Cu at (32.0, 102.0)
- added R107: 10k, Resistor_SMD:R_0603_1608Metric_Pad0.98x0.95mm_HandSolder, F.Cu at (64.0, 131.0)
- added R108: 10k, Resistor_SMD:R_0603_1608Metric_Pad0.98x0.95mm_HandSolder, F.Cu at (82.0, 131.0)
- added R109: 4.7k, Resistor_SMD:R_0603_1608Metric_Pad0.98x0.95mm_HandSolder, F.Cu at (37.0, 102.0)
- added R110: 150R, Resistor_SMD:R_0603_1608Metric_Pad0.98x0.95mm_HandSolder, F.Cu at (28.0, 141.0)
- added R111: 10k, Resistor_SMD:R_0603_1608Metric_Pad0.98x0.95mm_HandSolder, F.Cu at (27.0, 152.0)
- added R112: 33R, Resistor_SMD:R_0603_1608Metric_Pad0.98x0.95mm_HandSolder, F.Cu at (103.0, 117.0)
- added R113: 82R, Resistor_SMD:R_0603_1608Metric_Pad0.98x0.95mm_HandSolder, F.Cu at (36.0, 114.0)
- added R114: 82R, Resistor_SMD:R_0603_1608Metric_Pad0.98x0.95mm_HandSolder, F.Cu at (30.0, 114.5)
- added R115: 120R, Resistor_SMD:R_0603_1608Metric_Pad0.98x0.95mm_HandSolder, F.Cu at (27.0, 159.0)
- added R201: 1.2k, Resistor_SMD:R_0603_1608Metric_Pad0.98x0.95mm_HandSolder, F.Cu at (133.0, 109.0)
- added R202: 10k, Resistor_SMD:R_0603_1608Metric_Pad0.98x0.95mm_HandSolder, F.Cu at (133.0, 114.0)
- added R203: 62k, Resistor_SMD:R_0603_1608Metric_Pad0.98x0.95mm_HandSolder, F.Cu at (68.0, 179.0)
- added R204: 3.6k, Resistor_SMD:R_0603_1608Metric_Pad0.98x0.95mm_HandSolder, F.Cu at (68.0, 175.0)
- added R301: 10k, Resistor_SMD:R_0603_1608Metric_Pad0.98x0.95mm_HandSolder, F.Cu at (73.0, 178.0)
- added R302: 10k, Resistor_SMD:R_0603_1608Metric_Pad0.98x0.95mm_HandSolder, F.Cu at (73.0, 174.0)
- added R303: 22R, Resistor_SMD:R_0603_1608Metric_Pad0.98x0.95mm_HandSolder, F.Cu at (47.0, 127.0)
- added R304: 22R, Resistor_SMD:R_0603_1608Metric_Pad0.98x0.95mm_HandSolder, F.Cu at (47.0, 131.0)
- added R305: 1.5k, Resistor_SMD:R_0603_1608Metric_Pad0.98x0.95mm_HandSolder, F.Cu at (47.0, 137.0)
- added R306: 9.1k, Resistor_SMD:R_0603_1608Metric_Pad0.98x0.95mm_HandSolder, F.Cu at (47.0, 142.0)
- added R307: 4.7k, Resistor_SMD:R_0603_1608Metric_Pad0.98x0.95mm_HandSolder, F.Cu at (42.0, 142.0)
- added R308: 62k, Resistor_SMD:R_0603_1608Metric_Pad0.98x0.95mm_HandSolder, F.Cu at (28.0, 167.3)
- added R309: 62k, Resistor_SMD:R_0603_1608Metric_Pad0.98x0.95mm_HandSolder, F.Cu at (28.0, 171.3)
- added R401: 10k, Resistor_SMD:R_0603_1608Metric_Pad0.98x0.95mm_HandSolder, F.Cu at (68.0, 141.0)
- added R402: 4.7R, Resistor_SMD:R_0603_1608Metric_Pad0.98x0.95mm_HandSolder, F.Cu at (34.1, 35.0)
- added R403: 4.7R, Resistor_SMD:R_0603_1608Metric_Pad0.98x0.95mm_HandSolder, F.Cu at (37.0, 54.5)
- added R404: 4.7R, Resistor_SMD:R_0603_1608Metric_Pad0.98x0.95mm_HandSolder, F.Cu at (37.0, 71.5)
- added R405: 4.7R, Resistor_SMD:R_0603_1608Metric_Pad0.98x0.95mm_HandSolder, F.Cu at (37.0, 93.5)
- added R406: 33k, Resistor_SMD:R_0603_1608Metric_Pad0.98x0.95mm_HandSolder, F.Cu at (21.0, 61.5)
- added R407: 33k, Resistor_SMD:R_0603_1608Metric_Pad0.98x0.95mm_HandSolder, F.Cu at (118.0, 62.0)
- added R408: 10k, Resistor_SMD:R_0603_1608Metric_Pad0.98x0.95mm_HandSolder, F.Cu at (74.0, 141.0)
- added R409: 4.7R, Resistor_SMD:R_0603_1608Metric_Pad0.98x0.95mm_HandSolder, F.Cu at (106.9, 35.0)
- added R410: 4.7R, Resistor_SMD:R_0603_1608Metric_Pad0.98x0.95mm_HandSolder, F.Cu at (105.0, 55.0)
- added R411: 4.7R, Resistor_SMD:R_0603_1608Metric_Pad0.98x0.95mm_HandSolder, F.Cu at (104.0, 72.0)
- added R412: 4.7R, Resistor_SMD:R_0603_1608Metric_Pad0.98x0.95mm_HandSolder, F.Cu at (104.0, 94.0)
- added R501: 150R, Resistor_SMD:R_0603_1608Metric_Pad0.98x0.95mm_HandSolder, F.Cu at (86.8, 181.2)
- added R502: 150R, Resistor_SMD:R_0603_1608Metric_Pad0.98x0.95mm_HandSolder, F.Cu at (86.8, 177.2)
- added R503: 62k, Resistor_SMD:R_0603_1608Metric_Pad0.98x0.95mm_HandSolder, F.Cu at (86.8, 186.2)
- added R504: 62k, Resistor_SMD:R_0603_1608Metric_Pad0.98x0.95mm_HandSolder, F.Cu at (86.8, 190.2)
- added R505: 150R, Resistor_SMD:R_0603_1608Metric_Pad0.98x0.95mm_HandSolder, F.Cu at (86.0, 160.0)
- added R506: 150R, Resistor_SMD:R_0603_1608Metric_Pad0.98x0.95mm_HandSolder, F.Cu at (86.0, 164.0)
- added R507: 62k, Resistor_SMD:R_0603_1608Metric_Pad0.98x0.95mm_HandSolder, F.Cu at (86.0, 168.0)
- added R508: 62k, Resistor_SMD:R_0603_1608Metric_Pad0.98x0.95mm_HandSolder, F.Cu at (86.0, 172.0)
- added SW301: SW_Push, Button_Switch_SMD:SW_SPST_TL3342, F.Cu at (58.0, 161.0)
- added TH401: NTSA3104HZ048, Resistor_THT:R_Axial_DIN0309_L9.0mm_D3.2mm_P2.54mm_Vertical, F.Cu at (31.0, 64.1)
- added TH402: NTSA3104HZ048, Resistor_THT:R_Axial_DIN0309_L9.0mm_D3.2mm_P2.54mm_Vertical, F.Cu at (110.0, 64.5)
- added TP201: GND, TestPoint:TestPoint_Pad_D2.0mm, F.Cu at (129.0, 67.0)
- added TP202: +BATT, TestPoint:TestPoint_Pad_D2.0mm, F.Cu at (128.0, 61.0)
- added TP203: +3V3, TestPoint:TestPoint_Pad_D2.0mm, F.Cu at (136.0, 66.0)
- added TP204: +12V, TestPoint:TestPoint_Pad_D2.0mm, F.Cu at (135.0, 60.0)
- added U101: SN65HVD231DR, Package_SO:SOIC-8_3.9x4.9mm_P1.27mm, F.Cu at (33.5, 154.1)
- added U201: LM2596HVGT-ADJ, Package_TO_SOT_THT:TO-220-5_Vertical, F.Cu at (110.9, 115.4)
- added U202: XL1509-3.3E1, Package_SO:SOP-8_3.76x4.96mm_P1.27mm, F.Cu at (112.5, 134.9)
- added U301: STM32F103C8Tx, Package_QFP:LQFP-48_7x7mm_P0.5mm, F.Cu at (71.0, 150.0)
- added U302: M95640-WMN6TP, Package_SO:SOIC-8_3.9x4.9mm_P1.27mm, F.Cu at (35.5, 169.4)
- added U401: LM5110-1MX, Package_SO:SOIC-8_3.9x4.9mm_P1.27mm, F.Cu at (37.5, 43.6)
- added U402: LM5110-1MX, Package_SO:SOIC-8_3.9x4.9mm_P1.27mm, F.Cu at (37.5, 82.9)
- added U403: LM5110-1MX, Package_SO:SOIC-8_3.9x4.9mm_P1.27mm, F.Cu at (103.5, 43.9)
- added U404: LM5110-1MX, Package_SO:SOIC-8_3.9x4.9mm_P1.27mm, F.Cu at (103.5, 82.9)
- added Y301: 12MHz, Crystal:Crystal_SMD_3225-4Pin_3.2x2.5mm_HandSoldering, F.Cu at (61.5, 149.2)
Routing:
- added copper zone on B.Cu, net (none)
- added copper zone on F.Cu, net (none)
- added copper zone on B.Cu, net +BATT
- added copper zone on F.Cu, net GND
Other:
- board outline added: 91.1 x 100 mm
- copper layers 0 -> 4

Commit message: First PCB commit
Parts:
- removed U302: M95640-WMN6TP, Package_SO:SOIC-8_3.9x4.9mm_P1.27mm
- added C221: 100nF, Capacitor_SMD:C_0603_1608Metric_Pad1.08x0.95mm_HandSolder, F.Cu at (57.0, 172.0)
- added C222: 10nF, Capacitor_SMD:C_0603_1608Metric_Pad1.08x0.95mm_HandSolder, F.Cu at (58.0, 163.0)
- added C223: 100nF, Capacitor_SMD:C_0603_1608Metric_Pad1.08x0.95mm_HandSolder, F.Cu at (57.0, 175.0)
- added C224: 4.7uF, Capacitor_SMD:C_0603_1608Metric_Pad1.08x0.95mm_HandSolder, F.Cu at (57.0, 178.0)
- added C411: 1uF, Capacitor_SMD:C_0603_1608Metric_Pad1.08x0.95mm_HandSolder, F.Cu at (119.0, 79.0)
- added C412: 100nF, Capacitor_SMD:C_0603_1608Metric_Pad1.08x0.95mm_HandSolder, F.Cu at (119.0, 87.0)
- added C413: 1uF, Capacitor_SMD:C_0603_1608Metric_Pad1.08x0.95mm_HandSolder, F.Cu at (119.0, 112.0)
- added C414: 100nF, Capacitor_SMD:C_0603_1608Metric_Pad1.08x0.95mm_HandSolder, F.Cu at (119.0, 120.0)
- added D405: G30C120CTW, Package_TO_SOT_THT:TO-220-3_Vertical, F.Cu at (128.0, 85.0)
- added D406: G30C120CTW, Package_TO_SOT_THT:TO-220-3_Vertical, F.Cu at (128.0, 118.0)
- added Q409: STP15810, Package_TO_SOT_THT:TO-220-3_Vertical, F.Cu at (128.0, 74.0)
- added Q410: STP15810, Package_TO_SOT_THT:TO-220-3_Vertical, F.Cu at (128.0, 96.0)
- added Q411: STP15810, Package_TO_SOT_THT:TO-220-3_Vertical, F.Cu at (128.0, 107.0)
- added Q412: STP15810, Package_TO_SOT_THT:TO-220-3_Vertical, F.Cu at (128.0, 129.0)
- added R413: 4.7R, Resistor_SMD:R_0603_1608Metric_Pad0.98x0.95mm_HandSolder, F.Cu at (123.0, 74.0)
- added R414: 4.7R, Resistor_SMD:R_0603_1608Metric_Pad0.98x0.95mm_HandSolder, F.Cu at (123.0, 95.0)
- added R415: 4.7R, Resistor_SMD:R_0603_1608Metric_Pad0.98x0.95mm_HandSolder, F.Cu at (123.0, 107.0)
- added R416: 4.7R, Resistor_SMD:R_0603_1608Metric_Pad0.98x0.95mm_HandSolder, F.Cu at (123.0, 128.0)
- added U203: STM32F103C8Tx, Package_QFP:LQFP-48_7x7mm_P0.5mm, F.Cu at (49.0, 161.0)
- added U405: LM5110-1MX, Package_SO:SOIC-8_3.9x4.9mm_P1.27mm, F.Cu at (119.0, 83.0)
- added U406: LM5110-1MX, Package_SO:SOIC-8_3.9x4.9mm_P1.27mm, F.Cu at (119.0, 116.0)
- C101, C203, C204, C218, C219, C301, C302, C303, C304, C409, C410: footprint Capacitor_SMD:C_0805_2012Metric_Pad1.18x1.45mm_HandSolder -> Capacitor_SMD:C_0603_1608Metric_Pad1.08x0.95mm_HandSolder
- C202: footprint Capacitor_SMD:CP_Elec_10x10 -> Capacitor_SMD:CP_Elec_8x10.5
- C205, C206, C207, C208: footprint Capacitor_THT:CP_Radial_D16.0mm_P7.50mm -> Capacitor_THT:CP_Radial_D18.0mm_P7.50mm
- C209: value 100nF -> 2200uF; footprint Capacitor_SMD:C_0805_2012Metric_Pad1.18x1.45mm_HandSolder -> Capacitor_THT:CP_Radial_D18.0mm_P7.50mm
- C210: value 1mF -> 2200uF; footprint Capacitor_THT:CP_Radial_D10.0mm_P5.00mm -> Capacitor_THT:CP_Radial_D18.0mm_P7.50mm
- C211: value 330uF -> 2200uF; footprint Capacitor_SMD:CP_Elec_6.3x5.4 -> Capacitor_THT:CP_Radial_D18.0mm_P7.50mm
- C212: value 1nF -> 2200uF; footprint Capacitor_SMD:C_0805_2012Metric_Pad1.18x1.45mm_HandSolder -> Capacitor_THT:CP_Radial_D18.0mm_P7.50mm
- C213, C403, C407: value 1uF -> 100nF; footprint Capacitor_SMD:C_0805_2012Metric_Pad1.18x1.45mm_HandSolder -> Capacitor_SMD:C_0603_1608Metric_Pad1.08x0.95mm_HandSolder
- C214: value 10nF -> 1000uF; footprint Capacitor_SMD:C_0805_2012Metric_Pad1.18x1.45mm_HandSolder -> Capacitor_SMD:CP_Elec_10x10.5
- C215: value 100nF -> 330uF; footprint Capacitor_SMD:C_0805_2012Metric_Pad1.18x1.45mm_HandSolder -> Capacitor_SMD:CP_Elec_6.3x5.4
- C216: value 100nF -> 1nF; footprint Capacitor_SMD:C_0805_2012Metric_Pad1.18x1.45mm_HandSolder -> Capacitor_SMD:C_0603_1608Metric_Pad1.08x0.95mm_HandSolder
- C217, C402, C404: value 100nF -> 1uF; footprint Capacitor_SMD:C_0805_2012Metric_Pad1.18x1.45mm_HandSolder -> Capacitor_SMD:C_0603_1608Metric_Pad1.08x0.95mm_HandSolder
- C220: value 4.7uF -> 100nF; footprint Capacitor_SMD:C_0805_2012Metric_Pad1.18x1.45mm_HandSolder -> Capacitor_SMD:C_0603_1608Metric_Pad1.08x0.95mm_HandSolder
- C401: value 1uF -> 10nF; footprint Capacitor_SMD:C_0805_2012Metric_Pad1.18x1.45mm_HandSolder -> Capacitor_SMD:C_0603_1608Metric_Pad1.08x0.95mm_HandSolder
- C405: value 10nF -> 100nF; footprint Capacitor_SMD:C_0805_2012Metric_Pad1.18x1.45mm_HandSolder -> Capacitor_SMD:C_0603_1608Metric_Pad1.08x0.95mm_HandSolder
- C406: value 10nF -> 1uF; footprint Capacitor_SMD:C_0805_2012Metric_Pad1.18x1.45mm_HandSolder -> Capacitor_SMD:C_0603_1608Metric_Pad1.08x0.95mm_HandSolder
- C408: value 100nF -> 10nF; footprint Capacitor_SMD:C_0805_2012Metric_Pad1.18x1.45mm_HandSolder -> Capacitor_SMD:C_0603_1608Metric_Pad1.08x0.95mm_HandSolder
- H101, H102, H103, H104: footprint MountingHole:MountingHole_4.3mm_M4 -> MountingHole:MountingHole_2.7mm_M2.5
- L201, L202: footprint Resistor_SMD:R_0805_2012Metric_Pad1.20x1.40mm_HandSolder -> GozLib:L_10.4x10.4_H4.8_Handsoldering
- L203: footprint Resistor_SMD:R_0805_2012Metric_Pad1.20x1.40mm_HandSolder -> Inductor_SMD:L_0805_2012Metric_Pad1.15x1.40mm_HandSolder
- R402, R409: value 4.7R -> 33k
- R406, R407: value 33k -> 4.7R
- R408: value 10k -> 4.7R
- R410: value 4.7R -> 10k
- U301: value STM32F103C8Tx -> M95640-WMN6TP; footprint Package_QFP:LQFP-48_7x7mm_P0.5mm -> Package_SO:SOIC-8_3.9x4.9mm_P1.27mm
- moved C202 141.7 mm to (149.0, 219.5), turned to 90 degrees
- moved R410 105.5 mm to (57.0, 149.0)
- moved D202 105.5 mm to (162.0, 225.0), turned to -90 degrees
- moved D403 103.2 mm to (32.0, 113.0), turned to -90 degrees
- moved Q405 103.2 mm to (32.0, 102.0), turned to -90 degrees
- moved Q406 103.2 mm to (32.0, 124.0), turned to -90 degrees
- moved U202 103.0 mm to (142.5, 233.5), turned to -90 degrees
- moved R112 101.0 mm to (103.5, 218.0)
- moved D101 101.0 mm to (103.5, 223.0)
- moved D102 101.0 mm to (35.5, 212.0)
- moved D103 101.0 mm to (31.5, 212.0)
- moved J101 101.0 mm to (44.5, 222.0)
- moved J102 101.0 mm to (58.5, 208.0)
- moved J103 101.0 mm to (63.5, 222.5)
- moved J104 101.0 mm to (82.0, 222.5)
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Connections:
- C209 pad 1: +12V -> +BATT
- C210 pad 1: +12V -> +BATT
- C211 pad 1: +3V3 -> +BATT
- C212 pad 1: Net-(C212-Pad1) -> +BATT
- C212 pad 2: +12V -> GND
- C213 pad 1: +3.3VA -> +12V
- C214 pad 1: +3.3VA -> +12V
- C215 pad 1: GND -> +3V3
- C215 pad 2: +3V3 -> GND
- C216 pad 1: +3V3 -> Net-(C216-Pad1)
- C216 pad 2: GND -> +12V
- C217 pad 1: +3V3 -> +3.3VA
- C218 pad 1: /MCU/SUPPLY_MONITOR -> +3.3VA
- C219 pad 1: +3V3 -> GND
- C219 pad 2: GND -> +3V3
- C401 pad 1: GND -> /MCU/TEMP_LEFT
- C401 pad 2: +12V -> GND
- C405 pad 1: /MCU/TEMP_LEFT -> GND
- C405 pad 2: GND -> +12V
- C406 pad 1: /MCU/TEMP_RIGHT -> GND
- C406 pad 2: GND -> +12V
- C408 pad 1: GND -> /MCU/TEMP_RIGHT
- C408 pad 2: +12V -> GND
- D403 pad 1: /Motor driver/MOTOR_RIGHT -> /Motor driver/MOTOR_LEFT
- D403 pad 3: /Motor driver/MOTOR_RIGHT -> /Motor driver/MOTOR_LEFT
- J108 pad 1: /Solenoid driver/DIRECTION_COIL1 -> /Solenoid driver/DIRECTION_COIL2
- J108 pad 2: /Solenoid driver/DIRECTION_COIL2 -> /Solenoid driver/DIRECTION_COIL1
- J109 pad 1: /Solenoid driver/ENABLE_LEFT_COIL -> /Solenoid driver/ENABLE_RIGHT_COIL
- J109 pad 2: /Solenoid driver/ENABLE_RIGHT_COIL -> /Solenoid driver/ENABLE_LEFT_COIL
- Q405 pad 2: /Motor driver/MOTOR_RIGHT -> /Motor driver/MOTOR_LEFT
- Q406 pad 2: /Motor driver/MOTOR_RIGHT -> /Motor driver/MOTOR_LEFT
- R201 pad 2: Net-(C212-Pad1) -> Net-(C216-Pad1)
- R202 pad 1: Net-(C212-Pad1) -> Net-(C216-Pad1)
- R402 pad 1: Net-(R402-Pad1) -> /MCU/TEMP_LEFT
- R402 pad 2: Net-(Q401-Pad1) -> GND
- R403 pad 1: Net-(Q402-Pad1) -> Net-(R403-Pad1)
- R403 pad 2: Net-(R403-Pad2) -> Net-(Q401-Pad1)
- R404 pad 1: Net-(R404-Pad1) -> Net-(Q402-Pad1)
- R404 pad 2: Net-(Q403-Pad1) -> Net-(R404-Pad2)
- R405 pad 1: Net-(Q404-Pad1) -> Net-(R405-Pad1)
- R405 pad 2: Net-(R405-Pad2) -> Net-(Q403-Pad1)
- R406 pad 1: /MCU/TEMP_LEFT -> Net-(Q404-Pad1)
- R406 pad 2: GND -> Net-(R406-Pad2)
- R407 pad 1: /MCU/TEMP_RIGHT -> Net-(R407-Pad1)
- R407 pad 2: GND -> Net-(Q405-Pad1)
- R408 pad 1: /MCU/PWM_RIGHT -> Net-(Q406-Pad1)
- R408 pad 2: GND -> Net-(R408-Pad2)
- R409 pad 1: Net-(R409-Pad1) -> /MCU/TEMP_RIGHT
- R409 pad 2: Net-(Q405-Pad1) -> GND
- R410 pad 1: Net-(Q406-Pad1) -> /MCU/PWM_RIGHT
- R410 pad 2: Net-(R410-Pad2) -> GND
- R502 pad 1: Net-(Q501-Pad4) -> /MCU/DIRECTION2
- R502 pad 2: /MCU/DIRECTION2 -> Net-(Q501-Pad4)
- U201 pad 4: Net-(C212-Pad1) -> Net-(C216-Pad1)
- U301 pad 1: +3V3 -> /MCU/CS
- U301 pad 2: /MCU/DIRECTION -> /MCU/MISO
- U301 pad 3: /MCU/STEER_LOCK_LEFT -> +3V3
- U301 pad 4: /MCU/STEER_LOCK_RIGHT -> GND
- U301 pad 5: Net-(C303-Pad1) -> /MCU/MOSI
- U301 pad 6: Net-(C302-Pad1) -> /MCU/SCK
- U301 pad 7: /MCU/~{RST} -> +3V3
- U301 pad 8: GND -> +3V3
- U401 pad 5: Net-(R403-Pad2) -> Net-(R403-Pad1)
- U401 pad 7: Net-(R402-Pad1) -> Net-(R404-Pad2)
- U402 pad 5: Net-(R405-Pad2) -> Net-(R405-Pad1)
- U402 pad 7: Net-(R404-Pad1) -> Net-(R406-Pad2)
- U403 pad 2: /MCU/PWM_RIGHT -> /MCU/PWM_LEFT
- U403 pad 4: /MCU/PWM_RIGHT -> /MCU/PWM_LEFT
- U403 pad 5: Net-(R410-Pad2) -> Net-(R407-Pad1)
- U403 pad 7: Net-(R409-Pad1) -> Net-(R408-Pad2)
Routing:
- net /Motor driver/MOTOR_LEFT: track 0.00 -> 252.3 mm
- net /Motor driver/MOTOR_RIGHT: track 0.00 -> 251.5 mm
- net /MCU/PWM_RIGHT: track 0.00 -> 161.6 mm, vias 0 -> 6
- net +12V: track 0.00 -> 161.4 mm, vias 0 -> 16
- net +BATT: track 0.00 -> 129.4 mm
- net /MCU/PWM_LEFT: track 0.00 -> 104.8 mm, vias 0 -> 6
- net GND: track 0.00 -> 104.3 mm, vias 0 -> 20
- net /MCU/TEMP_RIGHT: track 0.00 -> 85.0 mm, vias 0 -> 1
- net Net-(C201-Pad1): track 0.00 -> 29.0 mm
- net Net-(D203-Pad1): track 0.00 -> 18.5 mm
- net /MCU/TEMP_LEFT: track 0.00 -> 15.0 mm, vias 0 -> 1
- net Net-(R405-Pad1): track 0.00 -> 11.7 mm, vias 0 -> 2
- net Net-(R407-Pad1): track 0.00 -> 11.7 mm, vias 0 -> 2
- net Net-(R403-Pad1): track 0.00 -> 11.7 mm, vias 0 -> 2
- net Net-(C216-Pad1): track 0.00 -> 11.5 mm, vias 0 -> 1
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- added copper zone on In2.Cu, net +12V
- added copper zone on F.Cu, net +BATT
- added copper zone on B.Cu, net GND
- removed copper zone on B.Cu, net +BATT
- removed copper zone on F.Cu, net GND
Other:
- board size 91.1 x 100 mm -> 110 x 160 mm

Commit message: Finish regulator layout
Parts:
- added R116: 10k, Resistor_SMD:R_0603_1608Metric_Pad0.98x0.95mm_HandSolder, F.Cu at (68.0, 175.5)
- added TP101: VBUS, TestPoint:TestPoint_Pad_D2.0mm, F.Cu at (101.0, 156.0)
- C201: footprint Capacitor_SMD:CP_Elec_10x10.5 -> Capacitor_THT:CP_Radial_D8.0mm_P3.50mm
- C214: footprint Capacitor_SMD:CP_Elec_10x10.5 -> Capacitor_THT:CP_Radial_D10.0mm_P5.00mm
- moved C215 110.6 mm to (78.5, 136.5)
- moved D204 106.7 mm to (88.5, 148.0), turned to -90 degrees
- moved D202 102.5 mm to (100.5, 143.0)
- moved C202 101.3 mm to (91.0, 136.5), turned to 180 degrees
- moved C204 99.9 mm to (97.0, 146.0), turned to -90 degrees
- moved D201 99.8 mm to (100.5, 134.5)
- moved U202 98.8 mm to (93.0, 148.0)
- moved L202 88.8 mm to (79.0, 149.0), turned to -90 degrees
- moved D101 87.3 mm to (30.5, 175.0), turned to 90 degrees
- moved R112 82.2 mm to (33.5, 175.0)
- moved R401 79.1 mm to (67.0, 230.5)
- moved R410 78.6 mm to (67.0, 227.0)
- moved R306 75.5 mm to (45.5, 167.5)
- moved C222 72.7 mm to (81.0, 232.0)
- moved R203 72.7 mm to (81.0, 226.0)
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Connections:
- U203 pad 10: /MCU/DIRECTION1 -> /MCU/ENABLE_RIGHT
- U203 pad 11: /MCU/DIRECTION2 -> /MCU/ENABLE_LEFT
- U203 pad 21: /MCU/ENABLE_LEFT -> /MCU/DIRECTION1
- U203 pad 22: /MCU/ENABLE_RIGHT -> /MCU/DIRECTION2
Routing:
- net +3V3: track 8.49 -> 278.7 mm, vias 0 -> 10
- net VBUS: track 0.00 -> 149.4 mm, vias 0 -> 3
- net GND: track 104.3 -> 220.7 mm, vias 20 -> 41
- net /MCU/ENABLE_LEFT: track 0.00 -> 68.9 mm, vias 0 -> 2
- net /MCU/ENABLE_RIGHT: track 0.00 -> 63.0 mm, vias 0 -> 2
- net /MCU/TEMP_LEFT: track 15.0 -> 76.9 mm
- net /MCU/DIRECTION1: track 0.00 -> 55.3 mm, vias 0 -> 2
- net /MCU/TEMP_RIGHT: track 85.0 -> 139.0 mm
- net /MCU/DIRECTION2: track 0.00 -> 51.8 mm, vias 0 -> 2
- net Net-(C202-Pad1): track 0.00 -> 20.8 mm
- net Net-(D204-Pad1): track 0.00 -> 20.4 mm
- net Net-(C303-Pad1): track 0.00 -> 16.5 mm
- net /MCU/BEEP: track 0.00 -> 15.4 mm
- net Net-(J110-Pad1): track 0.00 -> 14.9 mm
- net +12V: track 161.4 -> 175.1 mm, vias 16 -> 12
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- added copper zone on In2.Cu, net +3V3

Commit message: Finish PCB
Parts:
- added H111: MountingHole_Pad, MountingHole:MountingHole_4.3mm_M4_Pad, F.Cu at (54.5, 91.0)
- added H112: MountingHole_Pad, MountingHole:MountingHole_4.3mm_M4_Pad, F.Cu at (105.5, 91.0)
- moved C222 108.8 mm to (44.5, 129.5), turned to 90 degrees
- moved R204 106.7 mm to (42.5, 129.5), turned to 90 degrees
- moved R203 104.7 mm to (40.5, 129.5), turned to -90 degrees
- moved R401 98.5 mm to (45.0, 134.5)
- moved R410 94.2 mm to (49.0, 134.5), turned to 180 degrees
- moved C218 84.2 mm to (62.5, 149.0), turned to -90 degrees
- moved C217 81.9 mm to (60.5, 149.0), turned to -90 degrees
- moved R302 81.6 mm to (49.0, 163.0), turned to 180 degrees
- moved C301 80.4 mm to (59.5, 141.5)
- moved C219 80.3 mm to (61.0, 156.5), turned to 90 degrees
- moved R301 79.9 mm to (64.5, 141.5), turned to 180 degrees
- moved SW301 79.3 mm to (62.0, 137.5)
- moved R103 66.9 mm to (35.5, 171.5), turned to 90 degrees
- moved R305 66.8 mm to (41.5, 171.5), turned to 90 degrees
- moved R102 61.5 mm to (43.5, 171.5), turned to 90 degrees
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Connections:
- net /MCU/USB_DM renamed /MCU/USB_DN
- net Net-(R303-Pad1) renamed /MCU/D-
- net Net-(R304-Pad1) renamed /MCU/D+
- J107 pad 1: /MCU/SCK -> /MCU/MOSI
- J107 pad 3: /MCU/MOSI -> /MCU/SCK
- U203 pad 10: /MCU/ENABLE_RIGHT -> /MCU/DIRECTION1
- U203 pad 11: /MCU/ENABLE_LEFT -> /MCU/DIRECTION2
- U203 pad 14: /MCU/TEMP_LEFT -> /MCU/TEMP_RIGHT
- U203 pad 15: /MCU/TEMP_RIGHT -> /MCU/TEMP_LEFT
- U203 pad 16: /MCU/IO1 -> /MCU/IO3
- U203 pad 18: /MCU/IO3 -> /MCU/IO1
- U203 pad 2: /MCU/DIRECTION -> /MCU/STEER_LOCK_RIGHT
- U203 pad 21: /MCU/DIRECTION1 -> /MCU/ENABLE_LEFT
- U203 pad 22: /MCU/DIRECTION2 -> /MCU/ENABLE_RIGHT
- U203 pad 29: /MCU/PWM_LEFT -> /MCU/PWM_RIGHT
- U203 pad 31: /MCU/PWM_RIGHT -> /MCU/PWM_LEFT
- U203 pad 4: /MCU/STEER_LOCK_RIGHT -> /MCU/DIRECTION
Routing:
- net /MCU/~{RST}: track 0.00 -> 61.3 mm, vias 0 -> 2
- net /MCU/IGNITION: track 5.09 -> 61.5 mm, vias 0 -> 2
- net /MCU/DIRECTION: track 5.09 -> 59.8 mm
- net /MCU/TRACESWO: track 0.00 -> 49.1 mm, vias 0 -> 1
- net /MCU/THROTTLE: track 5.09 -> 46.6 mm, vias 0 -> 2
- net /MCU/SWCLK: track 0.00 -> 39.4 mm, vias 0 -> 1
- net /MCU/STEER_LOCK_RIGHT: track 5.06 -> 42.8 mm
- net GND: track 220.7 -> 257.6 mm, vias 41 -> 54
- net /MCU/SUPPLY_MONITOR: track 0.00 -> 36.4 mm
- net /MCU/SWDIO: track 0.00 -> 36.4 mm, vias 0 -> 1
- net /MCU/UART_RX: track 0.00 -> 32.9 mm, vias 0 -> 1
- net /MCU/PWM_LEFT: track 105.8 -> 138.2 mm, vias 6 -> 8
- net /MCU/IO1: track 0.00 -> 30.8 mm
- net /MCU/IO2: track 0.00 -> 30.7 mm
- net /MCU/IO3: track 0.00 -> 30.5 mm
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Other:
- board text added: "+12V"
- board text added: "+3V3"
- board text added: "+BATT"
- board text added: "3V3"
- board text added: "CAN"
- board text added: "CLK"
- board text added: "DIO"
- board text added: "DIR COIL"
- board text added: "ENABLE COIL"
- board text added: "FUSE"
- board text added: "G"
- board text added: "GND"
- board text added: "IGN/DIR"
- board text added: "JLCJLCJLCJLC"
- board text added: "LED1"
- board text added: "LED2"
- board text added: "LEFT"
- board text added: "PWR"
- board text added: "R"
- board text added: "RESET"
- board text added: "RIGHT"
- board text added: "RST"
- board text added: "STEER"
- board text added: "T"
- board text added: "THRTL"
- board text added: "TRC"
- board text added: "VBUS"
