File: motorcontroller.kicad_sch (KiCad schematic)
At the start: 48 parts, among them J101 TYPE-C-31-M-12, J102 STLink_02x05, J103 STRLCK, J104 IGN, J105 THROTTLE, J106 UART, J107 IO, J108 DIR, J109 EN, J110 CAN, Q101 AP2300, U101 SN65HVD231DR

Commit message: M3 mounting holes
Parts:
- H101, H102, H103, H104: footprint MountingHole:MountingHole_2.7mm_M2.5 -> MountingHole:MountingHole_3.2mm_M3
Changed lines of the file:
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@@
       (effects (font (size 1.27 1.27)) (justify left))
     )
-    (property "Footprint" "MountingHole:MountingHole_2.7mm_M2.5" (id 2) (at 21.59 184.15 0)
+    (property "Footprint" "MountingHole:MountingHole_3.2mm_M3" (id 2) (at 21.59 184.15 0)
       (effects (font (size 1.27 1.27)) hide)
     )
@@
       (effects (font (size 1.27 1.27)) (justify left))
     )
-    (property "Footprint" "MountingHole:MountingHole_2.7mm_M2.5" (id 2) (at 21.59 191.77 0)
+    (property "Footprint" "MountingHole:MountingHole_3.2mm_M3" (id 2) (at 21.59 191.77 0)
       (effects (font (size 1.27 1.27)) hide)
     )
@@
       (effects (font (size 1.27 1.27)) (justify left))
     )
-    (property "Footprint" "MountingHole:MountingHole_2.7mm_M2.5" (id 2) (at 43.18 184.15 0)
+    (property "Footprint" "MountingHole:MountingHole_3.2mm_M3" (id 2) (at 43.18 184.15 0)
       (effects (font (size 1.27 1.27)) hide)
     )
@@
       (effects (font (size 1.27 1.27)) (justify left))
     )
-    (property "Footprint" "MountingHole:MountingHole_2.7mm_M2.5" (id 2) (at 43.18 191.77 0)
+    (property "Footprint" "MountingHole:MountingHole_3.2mm_M3" (id 2) (at 43.18 191.77 0)
       (effects (font (size 1.27 1.27)) hide)
     )
@@
     )
     (path "/87f7301e-1686-425a-ae8e-c606aa1b298c"
-      (reference "H101") (unit 1) (value "MountingHole") (footprint "MountingHole:MountingHole_2.7mm_M2.5")
+      (reference "H101") (unit 1) (value "MountingHole") (footprint "MountingHole:MountingHole_3.2mm_M3")
     )
     (path "/60344553-e766-4e37-9e6d-ac8400813cf8"
-      (reference "H102") (unit 1) (value "MountingHole") (footprint "MountingHole:MountingHole_2.7mm_M2.5")
+      (reference "H102") (unit 1) (value "MountingHole") (footprint "MountingHole:MountingHole_3.2mm_M3")
     )
     (path "/11a6ad24-4e4f-4eb8-9f57-72096e25501c"
-      (reference "H103") (unit 1) (value "MountingHole") (footprint "MountingHole:MountingHole_2.7mm_M2.5")
+      (reference "H103") (unit 1) (value "MountingHole") (footprint "MountingHole:MountingHole_3.2mm_M3")
     )
     (path "/b4b08e88-e9fe-4b1e-b144-65181d0b4e12"
-      (reference "H104") (unit 1) (value "MountingHole") (footprint "MountingHole:MountingHole_2.7mm_M2.5")
+      (reference "H104") (unit 1) (value "MountingHole") (footprint "MountingHole:MountingHole_3.2mm_M3")
     )
     (path "/494d5f8f-6ff7-44eb-9cb3-0995471395d8"

Commit message: Tweak PCB and add gerbers
Parts:
- added C102: 4.7nF, Capacitor_SMD:C_0603_1608Metric_Pad1.08x0.95mm_HandSolder, symbol Device:C
- added D104: NUP2105L, Package_TO_SOT_SMD:SOT-23, symbol Power_Protection:NUP2105L
- added D105: PRTR5V0U2X, Package_TO_SOT_SMD:SOT-143, symbol Power_Protection:PRTR5V0U2X
- added R117: 10k, Resistor_SMD:R_0603_1608Metric_Pad0.98x0.95mm_HandSolder, symbol Device:R
- added R118: 60R, Resistor_SMD:R_0603_1608Metric_Pad0.98x0.95mm_HandSolder, symbol Device:R
- added R119, R120, R121, R122: 22R, Resistor_SMD:R_0603_1608Metric_Pad0.98x0.95mm_HandSolder, symbol Device:R
- J101: footprint Connector_USB:USB_C_Receptacle_HRO_TYPE-C-31-M-12 -> GozLib:USB_C_Receptacle_HRO_TYPE-C-31-M-12_Handsoldering
- R115: value 120R -> 60R
Connections:
- net GND: now also C102.2, D104.3 (A), D105.1 (GND), R117.2
- net MCU/CAN_RX: now also R122.2; no longer U101.4 (RXD)
- net MCU/CAN_TX: now also R121.1; no longer U101.1 (TXD)
- net MCU/UART_RX: now also R119.2; no longer J106.3 (Pin_3), R106.2
- net MCU/UART_TX: now also R120.1; no longer J106.1 (Pin_1), R109.2
- net MCU/USB_DN: now also D105.2 (I/O1)
- net MCU/USB_DP: now also D105.3 (I/O2)
- net VBUS: now also D105.4 (VCC)
- net at Q101.1 (G), R110.2: now also R117.1
- net at U101.5 (Vref): now also R115.2, C102.1, R118.1
- net at R115.1, U101.7 (CANH): now also J110.3 (Pin_3), D104.1 (K); no longer J110.1 (Pin_1)
- new net: D104.2 (K), J110.1 (Pin_1), R118.2, U101.6 (CANL)
- new net: R121.2, U101.1 (TXD)
- new net: R122.1, U101.4 (RXD)
- new net: J106.3 (Pin_3), R106.2, R119.1
- new net: J106.1 (Pin_1), R109.2, R120.2
- no-connect marks 4 -> 3
Other:
- moved on the sheet: J101, J106, J110, R101, R102, R103, R106, R109, R115, TP101
