File: solenoiddriver.kicad_sch (KiCad schematic)
At the start: 16 parts

Commit message: Annotate schematic
Parts:
- gave numbers to parts that had none: 14
Changed lines of the file:
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@@
   (symbol (lib_id "power:+BATT") (at 100.33 29.21 0) (unit 1)
     (in_bom yes) (on_board yes) (fields_autoplaced)
-    (property "Reference" "#PWR?" (id 0) (at 100.33 33.02 0)
+    (property "Reference" "#PWR0503" (id 0) (at 100.33 33.02 0)
       (effects (font (size 1.27 1.27)) hide)
     )
@@
   (symbol (lib_id "power:+BATT") (at 100.33 60.96 0) (unit 1)
     (in_bom yes) (on_board yes) (fields_autoplaced)
-    (property "Reference" "#PWR?" (id 0) (at 100.33 64.77 0)
+    (property "Reference" "#PWR0504" (id 0) (at 100.33 64.77 0)
       (effects (font (size 1.27 1.27)) hide)
     )
@@
   (symbol (lib_id "power:+BATT") (at 185.42 29.21 0) (unit 1)
     (in_bom yes) (on_board yes) (fields_autoplaced)
-    (property "Reference" "#PWR?" (id 0) (at 185.42 33.02 0)
+    (property "Reference" "#PWR0507" (id 0) (at 185.42 33.02 0)
       (effects (font (size 1.27 1.27)) hide)
     )
@@
   (symbol (lib_id "power:+BATT") (at 185.42 60.96 0) (unit 1)
     (in_bom yes) (on_board yes) (fields_autoplaced)
-    (property "Reference" "#PWR?" (id 0) (at 185.42 64.77 0)
+    (property "Reference" "#PWR0508" (id 0) (at 185.42 64.77 0)
       (effects (font (size 1.27 1.27)) hide)
     )
@@
   (symbol (lib_id "power:GND") (at 81.28 58.42 0) (unit 1)
     (in_bom yes) (on_board yes) (fields_autoplaced)
-    (property "Reference" "#PWR?" (id 0) (at 81.28 64.77 0)
+    (property "Reference" "#PWR0501" (id 0) (at 81.28 64.77 0)
       (effects (font (size 1.27 1.27)) hide)
     )
@@
   (symbol (lib_id "power:GND") (at 81.28 90.17 0) (unit 1)
     (in_bom yes) (on_board yes) (fields_autoplaced)
-    (property "Reference" "#PWR?" (id 0) (at 81.28 96.52 0)
+    (property "Reference" "#PWR0502" (id 0) (at 81.28 96.52 0)
       (effects (font (size 1.27 1.27)) hide)
     )
@@
   (symbol (lib_id "power:GND") (at 166.37 58.42 0) (unit 1)
     (in_bom yes) (on_board yes) (fields_autoplaced)
-    (property "Reference" "#PWR?" (id 0) (at 166.37 64.77 0)
+    (property "Reference" "#PWR0505" (id 0) (at 166.37 64.77 0)
       (effects (font (size 1.27 1.27)) hide)
     )
@@
   (symbol (lib_id "power:GND") (at 166.37 90.17 0) (unit 1)
     (in_bom yes) (on_board yes) (fields_autoplaced)
-    (property "Reference" "#PWR?" (id 0) (at 166.37 96.52 0)
+    (property "Reference" "#PWR0506" (id 0) (at 166.37 96.52 0)
       (effects (font (size 1.27 1.27)) hide)
     )
@@
   (symbol (lib_id "Device:R") (at 64.77 46.99 90) (unit 1)
     (in_bom yes) (on_board yes)
-    (property "Reference" "R?" (id 0) (at 64.77 44.45 90))
+    (property "Reference" "R501" (id 0) (at 64.77 44.45 90))
     (property "Value" "150R" (id 1) (at 64.77 46.99 90))
     (property "Footprint" "" (id 2) (at 64.77 48.768 90)
@@
   (symbol (lib_id "Device:R") (at 64.77 78.74 270) (unit 1)
     (in_bom yes) (on_board yes)
-    (property "Reference" "R?" (id 0) (at 64.77 76.2 90))
+    (property "Reference" "R502" (id 0) (at 64.77 76.2 90))
     (property "Value" "150R" (id 1) (at 64.77 78.74 90))
     (property "Footprint" "" (id 2) (at 64.77 76.962 90)
@@
   (symbol (lib_id "Device:R") (at 71.12 52.07 0) (unit 1)
     (in_bom yes) (on_board yes)
-    (property "Reference" "R?" (id 0) (at 72.39 50.7999 0)
+    (property "Reference" "R503" (id 0) (at 72.39 50.7999 0)
       (effects (font (size 1.27 1.27)) (justify left))
     )
@@
   (symbol (lib_id "Device:R") (at 71.12 83.82 180) (unit 1)
     (in_bom yes) (on_board yes)
-    (property "Reference" "R?" (id 0) (at 72.39 82.5499 0)
+    (property "Reference" "R504" (id 0) (at 72.39 82.5499 0)
       (effects (font (size 1.27 1.27)) (justify right))
     )
@@
   (symbol (lib_id "Device:R") (at 149.86 46.99 90) (unit 1)
     (in_bom yes) (on_board yes)
-    (property "Reference" "R?" (id 0) (at 149.86 44.45 90))
+    (property "Reference" "R505" (id 0) (at 149.86 44.45 90))
     (property "Value" "150R" (id 1) (at 149.86 46.99 90))
     (property "Footprint" "" (id 2) (at 149.86 48.768 90)
@@
   (symbol (lib_id "Device:R") (at 149.86 78.74 90) (unit 1)
     (in_bom yes) (on_board yes)
-    (property "Reference" "R?" (id 0) (at 149.86 76.2 90))
+    (property "Reference" "R506" (id 0) (at 149.86 76.2 90))
     (property "Value" "150R" (id 1) (at 149.86 78.74 90))
     (property "Footprint" "" (id 2) (at 149.86 80.518 90)
@@
   (symbol (lib_id "Device:R") (at 156.21 52.07 0) (unit 1)
     (in_bom yes) (on_board yes)
-    (property "Reference" "R?" (id 0) (at 157.48 50.7999 0)
+    (property "Reference" "R507" (id 0) (at 157.48 50.7999 0)
       (effects (font (size 1.27 1.27)) (justify left))
     )
@@
   (symbol (lib_id "Device:R") (at 156.21 83.82 0) (unit 1)
     (in_bom yes) (on_board yes)
-    (property "Reference" "R?" (id 0) (at 157.48 82.5499 0)
+    (property "Reference" "R508" (id 0) (at 157.48 82.5499 0)
       (effects (font (size 1.27 1.27)) (justify left))
     )
@@
   (symbol (lib_id "Device:D_Schottky") (at 100.33 33.02 270) (unit 1)
     (in_bom yes) (on_board yes) (fields_autoplaced)
-    (property "Reference" "D?" (id 0) (at 102.87 31.7499 90)
+    (property "Reference" "D501" (id 0) (at 102.87 31.7499 90)
       (effects (font (size 1.27 1.27)) (justify left))
     )
@@
   (symbol (lib_id "Device:D_Schottky") (at 100.33 64.77 270) (unit 1)
     (in_bom yes) (on_board yes) (fields_autoplaced)
-    (property "Reference" "D?" (id 0) (at 102.87 63.4999 90)
+    (property "Reference" "D502" (id 0) (at 102.87 63.4999 90)
       (effects (font (size 1.27 1.27)) (justify left))
     )
@@
   (symbol (lib_id "Device:D_Schottky") (at 185.42 33.02 270) (unit 1)
     (in_bom yes) (on_board yes) (fields_autoplaced)
-    (property "Reference" "D?" (id 0) (at 187.96 31.7499 90)
+    (property "Reference" "D503" (id 0) (at 187.96 31.7499 90)
       (effects (font (size 1.27 1.27)) (justify left))
     )
@@
   (symbol (lib_id "Device:D_Schottky") (at 185.42 64.77 270) (unit 1)
     (in_bom yes) (on_board yes) (fields_autoplaced)
-    (property "Reference" "D?" (id 0) (at 187.96 63.4999 90)
+    (property "Reference" "D504" (id 0) (at 187.96 63.4999 90)
       (effects (font (size 1.27 1.27)) (justify left))
     )
@@
   (symbol (lib_id "GozLib:WSP6946") (at 78.74 46.99 0) (unit 1)
     (in_bom yes) (on_board yes) (fields_autoplaced)
-    (property "Reference" "Q?" (id 0) (at 85.09 45.7199 0)
+    (property "Reference" "Q501" (id 0) (at 85.09 45.7199 0)
       (effects (font (size 1.27 1.27)) (justify left))
     )
@@
   (symbol (lib_id "GozLib:WSP6946") (at 78.74 78.74 0) (unit 2)
     (in_bom yes) (on_board yes) (fields_autoplaced)
-    (property "Reference" "Q?" (id 0) (at 85.09 77.4699 0)
+    (property "Reference" "Q501" (id 0) (at 85.09 77.4699 0)
       (effects (font (size 1.27 1.27)) (justify left))
     )
@@
   (symbol (lib_id "GozLib:WSP6946") (at 163.83 46.99 0) (unit 1)
     (in_bom yes) (on_board yes) (fields_autoplaced)
-    (property "Reference" "Q?" (id 0) (at 170.18 45.7199 0)
+    (property "Reference" "Q502" (id 0) (at 170.18 45.7199 0)
       (effects (font (size 1.27 1.27)) (justify left))
     )
@@
   (symbol (lib_id "GozLib:WSP6946") (at 163.83 78.74 0) (unit 2)
     (in_bom yes) (on_board yes) (fields_autoplaced)
-    (property "Reference" "Q?" (id 0) (at 170.18 77.4699 0)
-      (effects (font (size 1.27 1.27)) (justify left))
-    )
+    (property "Reference" "Q502" (id 0) (at 170.18 77.4699 0)
+      (effects (font (size 1.27 1.27)) (justify left))
+    )

Commit message: Clean up BOM
Parts:
- R503, R504, R507, R508: value 62K -> 62k
Changed lines of the file:
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@@
       (effects (font (size 1.27 1.27)) (justify left))
     )
-    (property "Value" "62K" (id 1) (at 72.39 53.3399 0)
+    (property "Value" "62k" (id 1) (at 72.39 53.3399 0)
       (effects (font (size 1.27 1.27)) (justify left))
     )
@@
       (effects (font (size 1.27 1.27)) (justify right))
     )
-    (property "Value" "62K" (id 1) (at 72.39 85.0899 0)
+    (property "Value" "62k" (id 1) (at 72.39 85.0899 0)
       (effects (font (size 1.27 1.27)) (justify right))
     )
@@
       (effects (font (size 1.27 1.27)) (justify left))
     )
-    (property "Value" "62K" (id 1) (at 157.48 53.3399 0)
+    (property "Value" "62k" (id 1) (at 157.48 53.3399 0)
       (effects (font (size 1.27 1.27)) (justify left))
     )
@@
       (effects (font (size 1.27 1.27)) (justify left))
     )
-    (property "Value" "62K" (id 1) (at 157.48 85.0899 0)
+    (property "Value" "62k" (id 1) (at 157.48 85.0899 0)
       (effects (font (size 1.27 1.27)) (justify left))
     )

Commit message: Assign footprints
Parts:
- D501, D502, D503, D504: footprint (none) -> Diode_SMD:D_SMA_Handsoldering
- R501, R502, R503, R504, R505, R506, R507, R508: footprint (none) -> Resistor_SMD:R_0805_2012Metric_Pad1.20x1.40mm_HandSolder
Changed lines of the file:
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@@
     (property "Reference" "R501" (id 0) (at 64.77 44.45 90))
     (property "Value" "150R" (id 1) (at 64.77 46.99 90))
-    (property "Footprint" "" (id 2) (at 64.77 48.768 90)
+    (property "Footprint" "Resistor_SMD:R_0805_2012Metric_Pad1.20x1.40mm_HandSolder" (id 2) (at 64.77 48.768 90)
       (effects (font (size 1.27 1.27)) hide)
     )
@@
     (property "Reference" "R502" (id 0) (at 64.77 76.2 90))
     (property "Value" "150R" (id 1) (at 64.77 78.74 90))
-    (property "Footprint" "" (id 2) (at 64.77 76.962 90)
+    (property "Footprint" "Resistor_SMD:R_0805_2012Metric_Pad1.20x1.40mm_HandSolder" (id 2) (at 64.77 76.962 90)
       (effects (font (size 1.27 1.27)) hide)
     )
@@
       (effects (font (size 1.27 1.27)) (justify left))
     )
-    (property "Footprint" "" (id 2) (at 69.342 52.07 90)
+    (property "Footprint" "Resistor_SMD:R_0805_2012Metric_Pad1.20x1.40mm_HandSolder" (id 2) (at 69.342 52.07 90)
       (effects (font (size 1.27 1.27)) hide)
     )
@@
       (effects (font (size 1.27 1.27)) (justify right))
     )
-    (property "Footprint" "" (id 2) (at 72.898 83.82 90)
+    (property "Footprint" "Resistor_SMD:R_0805_2012Metric_Pad1.20x1.40mm_HandSolder" (id 2) (at 72.898 83.82 90)
       (effects (font (size 1.27 1.27)) hide)
     )
@@
     (property "Reference" "R505" (id 0) (at 149.86 44.45 90))
     (property "Value" "150R" (id 1) (at 149.86 46.99 90))
-    (property "Footprint" "" (id 2) (at 149.86 48.768 90)
+    (property "Footprint" "Resistor_SMD:R_0805_2012Metric_Pad1.20x1.40mm_HandSolder" (id 2) (at 149.86 48.768 90)
       (effects (font (size 1.27 1.27)) hide)
     )
@@
     (property "Reference" "R506" (id 0) (at 149.86 76.2 90))
     (property "Value" "150R" (id 1) (at 149.86 78.74 90))
-    (property "Footprint" "" (id 2) (at 149.86 80.518 90)
+    (property "Footprint" "Resistor_SMD:R_0805_2012Metric_Pad1.20x1.40mm_HandSolder" (id 2) (at 149.86 80.518 90)
       (effects (font (size 1.27 1.27)) hide)
     )
@@
       (effects (font (size 1.27 1.27)) (justify left))
     )
-    (property "Footprint" "" (id 2) (at 154.432 52.07 90)
+    (property "Footprint" "Resistor_SMD:R_0805_2012Metric_Pad1.20x1.40mm_HandSolder" (id 2) (at 154.432 52.07 90)
       (effects (font (size 1.27 1.27)) hide)
     )
@@
       (effects (font (size 1.27 1.27)) (justify left))
     )
-    (property "Footprint" "" (id 2) (at 154.432 83.82 90)
+    (property "Footprint" "Resistor_SMD:R_0805_2012Metric_Pad1.20x1.40mm_HandSolder" (id 2) (at 154.432 83.82 90)
       (effects (font (size 1.27 1.27)) hide)
     )
@@
       (effects (font (size 1.27 1.27)) (justify left))
     )
-    (property "Footprint" "" (id 2) (at 100.33 33.02 0)
+    (property "Footprint" "Diode_SMD:D_SMA_Handsoldering" (id 2) (at 100.33 33.02 0)
       (effects (font (size 1.27 1.27)) hide)
     )
@@
       (effects (font (size 1.27 1.27)) (justify left))
     )
-    (property "Footprint" "" (id 2) (at 100.33 64.77 0)
+    (property "Footprint" "Diode_SMD:D_SMA_Handsoldering" (id 2) (at 100.33 64.77 0)
       (effects (font (size 1.27 1.27)) hide)
     )
@@
       (effects (font (size 1.27 1.27)) (justify left))
     )
-    (property "Footprint" "" (id 2) (at 185.42 33.02 0)
+    (property "Footprint" "Diode_SMD:D_SMA_Handsoldering" (id 2) (at 185.42 33.02 0)
       (effects (font (size 1.27 1.27)) hide)
     )
@@
       (effects (font (size 1.27 1.27)) (justify left))
     )
-    (property "Footprint" "" (id 2) (at 185.42 64.77 0)
+    (property "Footprint" "Diode_SMD:D_SMA_Handsoldering" (id 2) (at 185.42 64.77 0)
       (effects (font (size 1.27 1.27)) hide)
     )

Commit message: Start PCB
Parts:
- R501, R502, R503, R504, R505, R506, R507, R508: footprint Resistor_SMD:R_0805_2012Metric_Pad1.20x1.40mm_HandSolder -> Resistor_SMD:R_0603_1608Metric_Pad0.98x0.95mm_HandSolder
Changed lines of the file:
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@@
     (property "Reference" "R501" (id 0) (at 64.77 44.45 90))
     (property "Value" "150R" (id 1) (at 64.77 46.99 90))
-    (property "Footprint" "Resistor_SMD:R_0805_2012Metric_Pad1.20x1.40mm_HandSolder" (id 2) (at 64.77 48.768 90)
+    (property "Footprint" "Resistor_SMD:R_0603_1608Metric_Pad0.98x0.95mm_HandSolder" (id 2) (at 64.77 48.768 90)
       (effects (font (size 1.27 1.27)) hide)
     )
@@
     (property "Reference" "R502" (id 0) (at 64.77 76.2 90))
     (property "Value" "150R" (id 1) (at 64.77 78.74 90))
-    (property "Footprint" "Resistor_SMD:R_0805_2012Metric_Pad1.20x1.40mm_HandSolder" (id 2) (at 64.77 76.962 90)
+    (property "Footprint" "Resistor_SMD:R_0603_1608Metric_Pad0.98x0.95mm_HandSolder" (id 2) (at 64.77 76.962 90)
       (effects (font (size 1.27 1.27)) hide)
     )
@@
       (effects (font (size 1.27 1.27)) (justify left))
     )
-    (property "Footprint" "Resistor_SMD:R_0805_2012Metric_Pad1.20x1.40mm_HandSolder" (id 2) (at 69.342 52.07 90)
+    (property "Footprint" "Resistor_SMD:R_0603_1608Metric_Pad0.98x0.95mm_HandSolder" (id 2) (at 69.342 52.07 90)
       (effects (font (size 1.27 1.27)) hide)
     )
@@
       (effects (font (size 1.27 1.27)) (justify right))
     )
-    (property "Footprint" "Resistor_SMD:R_0805_2012Metric_Pad1.20x1.40mm_HandSolder" (id 2) (at 72.898 83.82 90)
+    (property "Footprint" "Resistor_SMD:R_0603_1608Metric_Pad0.98x0.95mm_HandSolder" (id 2) (at 72.898 83.82 90)
       (effects (font (size 1.27 1.27)) hide)
     )
@@
     (property "Reference" "R505" (id 0) (at 149.86 44.45 90))
     (property "Value" "150R" (id 1) (at 149.86 46.99 90))
-    (property "Footprint" "Resistor_SMD:R_0805_2012Metric_Pad1.20x1.40mm_HandSolder" (id 2) (at 149.86 48.768 90)
+    (property "Footprint" "Resistor_SMD:R_0603_1608Metric_Pad0.98x0.95mm_HandSolder" (id 2) (at 149.86 48.768 90)
       (effects (font (size 1.27 1.27)) hide)
     )
@@
     (property "Reference" "R506" (id 0) (at 149.86 76.2 90))
     (property "Value" "150R" (id 1) (at 149.86 78.74 90))
-    (property "Footprint" "Resistor_SMD:R_0805_2012Metric_Pad1.20x1.40mm_HandSolder" (id 2) (at 149.86 80.518 90)
+    (property "Footprint" "Resistor_SMD:R_0603_1608Metric_Pad0.98x0.95mm_HandSolder" (id 2) (at 149.86 80.518 90)
       (effects (font (size 1.27 1.27)) hide)
     )
@@
       (effects (font (size 1.27 1.27)) (justify left))
     )
-    (property "Footprint" "Resistor_SMD:R_0805_2012Metric_Pad1.20x1.40mm_HandSolder" (id 2) (at 154.432 52.07 90)
+    (property "Footprint" "Resistor_SMD:R_0603_1608Metric_Pad0.98x0.95mm_HandSolder" (id 2) (at 154.432 52.07 90)
       (effects (font (size 1.27 1.27)) hide)
     )
@@
       (effects (font (size 1.27 1.27)) (justify left))
     )
-    (property "Footprint" "Resistor_SMD:R_0805_2012Metric_Pad1.20x1.40mm_HandSolder" (id 2) (at 154.432 83.82 90)
+    (property "Footprint" "Resistor_SMD:R_0603_1608Metric_Pad0.98x0.95mm_HandSolder" (id 2) (at 154.432 83.82 90)
       (effects (font (size 1.27 1.27)) hide)
     )

Commit message: Finish regulator layout
Connections:
- net DIRECTION_IN2: now also R502.1; no longer R502.2
- net at Q501.4 (G), R504.2: now also R502.2; no longer R502.1
Other:
- moved on the sheet: R502
Changed lines of the file:
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@@
     (pin "2")
   )
-  (symbol (lib_id "Device:R") (at 64.77 78.74 270) (unit 1)
+  (symbol (lib_id "Device:R") (at 64.77 78.74 90) (unit 1)
     (in_bom yes) (on_board yes)
     (property "Reference" "R502" (id 0) (at 64.77 76.2 90))
     (property "Value" "150R" (id 1) (at 64.77 78.74 90))
-    (property "Footprint" "Resistor_SMD:R_0603_1608Metric_Pad0.98x0.95mm_HandSolder" (id 2) (at 64.77 76.962 90)
+    (property "Footprint" "Resistor_SMD:R_0603_1608Metric_Pad0.98x0.95mm_HandSolder" (id 2) (at 64.77 80.518 90)
       (effects (font (size 1.27 1.27)) hide)
     )

Commit message: Tweak PCB and add gerbers
Parts:
- R503, R504, R507, R508: value 62k -> 10k
Changed lines of the file:
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@@
       (effects (font (size 1.27 1.27)) (justify left))
     )
-    (property "Value" "62k" (id 1) (at 72.39 53.3399 0)
+    (property "Value" "10k" (id 1) (at 72.39 53.3399 0)
       (effects (font (size 1.27 1.27)) (justify left))
     )
@@
       (effects (font (size 1.27 1.27)) (justify right))
     )
-    (property "Value" "62k" (id 1) (at 72.39 85.0899 0)
+    (property "Value" "10k" (id 1) (at 72.39 85.0899 0)
       (effects (font (size 1.27 1.27)) (justify right))
     )
@@
       (effects (font (size 1.27 1.27)) (justify left))
     )
-    (property "Value" "62k" (id 1) (at 157.48 53.3399 0)
+    (property "Value" "10k" (id 1) (at 157.48 53.3399 0)
       (effects (font (size 1.27 1.27)) (justify left))
     )
@@
       (effects (font (size 1.27 1.27)) (justify left))
     )
-    (property "Value" "62k" (id 1) (at 157.48 85.0899 0)
+    (property "Value" "10k" (id 1) (at 157.48 85.0899 0)
       (effects (font (size 1.27 1.27)) (justify left))
     )
